Commit message: upgrade

File: rover/urdf/camera.xacro (robot description, xacro)
@@ -24,5 +24,5 @@
       <child link="camera_link"/>
       <!-- <origin rpy="0 0 0" xyz="0.05 0 0.02"/> -->
-      <origin rpy="0 1.34 0" xyz="0.06 0 0.02"/>
+      <origin rpy="0 1.39626 0" xyz="0.07 0 0.02"/>
       <!-- <origin rpy="0 1.5708 0" xyz="0.077 0 0.028"/> -->
       <limit effort="30" velocity="1.0"/>
@@ -45,5 +45,5 @@
         <image>
           <width>800</width>
-          <height>800</height>
+          <height>500</height>
           <!-- <width>684</width>
           <height>456</height> -->

File: rover/urdf/robot.urdf.xacro (robot description, xacro)
@@ -45,5 +45,5 @@
   </joint>
   <gazebo reference="back_wheel">
-    <material>Gazebo/Blue</material>
+    <material>Gazebo/Black</material>
     <mu1>0.0</mu1>
     <mu2>0.0</mu2>
@@ -54,5 +54,5 @@
   </gazebo>
   <gazebo reference="base_link">
-    <material>Gazebo/White</material>
+    <material>Gazebo/Green</material>
     <mu1>0.0</mu1>
     <mu2>0.0</mu2>
@@ -60,5 +60,4 @@
     <gravity>true</gravity>
   </gazebo>
-  <!-- Add ROS plugin so we can interact with our robot -->
   <gazebo>
     <plugin name="gazebo_ros_control" filename="libgazebo_ros_control.so">
